File: KiCad Project/Tutorial.kicad_pcb (KiCad board)
At the start: 2 copper layers, 49.7 x 82.4 mm, 30 parts, among them J1 USB_mini_micro_B, K1 KEYSW, K2 KEYSW, K3 KEYSW, K4 KEYSW, K5 KEYSW, SW1 SW_PUSH, U1 ATMEGA32U4, Y2 16Mhz

Commit message: Added Fuse
Parts:
- added F1: 500mA, Fuse:Fuse_1206_3216Metric, B.Cu at (68.7, 42.9)
Connections:
- U1 pad 2: VCC -> Net-(F1-Pad1)
Routing:
- net VCC: track 89.7 -> 97.1 mm
- net Net-(F1-Pad1): track 0.00 -> 5.66 mm
